Commit message: A bunch of experimentation and setup done. AprilTags left out though.

File: simenv/urdf/belt.xacro (robot description, xacro)
@@ -1,7 +1,7 @@
 <?xml version="1.0" encoding="utf-8"?>
 <robot name="belt">
-  <link name="world"/>
+  <link name="virtualLink"/>
   <joint name="joint_fix" type="fixed">
-    <parent link="world"/>
+    <parent link="virtualLink"/>
     <child link="belt_base_link"/>
   </joint>
@@ -29,5 +29,5 @@
   </link>
   <joint name="dbelt_joint" type="planar">
-    <parent link = "world"/>
+    <parent link = "virtualLink"/>
     <child link = "dbelt" />
     <axis xyz="0 1 0"/>

Commit message: Final Commit to worthless design

File: simenv/urdf/belt.xacro (robot description, xacro)
@@ -1,9 +1,4 @@
 <?xml version="1.0" encoding="utf-8"?>
 <robot name="belt">
-  <link name="virtualLink"/>
-  <joint name="joint_fix" type="fixed">
-    <parent link="virtualLink"/>
-    <child link="belt_base_link"/>
-  </joint>
   <link name="belt_base_link">
     <collision>
@@ -29,5 +24,5 @@
   </link>
   <joint name="dbelt_joint" type="planar">
-    <parent link = "virtualLink"/>
+    <parent link = "belt_base_link"/>
     <child link = "dbelt" />
     <axis xyz="0 1 0"/>
@@ -35,4 +30,10 @@
   </joint>
   <link name="dbelt">
+    <visual>
+      <origin xyz="0 -4.25 -0.01" rpy="0 0 0"/>
+      <geometry>
+        <box size= "1.0 0.5 0.01"/>
+      </geometry>
+    </visual>
     <collision>
       <origin xyz="0 -4.25 -0.01" rpy="0 0 0"/>
@@ -59,3 +60,16 @@
     </plugin>
   </gazebo>
+  <gazebo reference="belt_base_link">
+    <mu1>30</mu1>
+    <mu2>30</mu2>
+    <kp>1000000</kp>
+    <kd>1</kd>
+    <static>1</static>
+  </gazebo>
+  <gazebo reference="dbelt">
+    <mu1>30</mu1>
+    <mu2>30</mu2>
+    <kp>1000000</kp>
+    <kd>1</kd>
+  </gazebo>
 </robot>

File: simenv/urdf/simenv.urdf (robot description, URDF)
Before this commit: robot lemons, 8 links, 7 joints
Links:
- link base_link: mass 100 -> 10000
